File: clock3.kicad_pcb (KiCad board)
At the start: 2 copper layers, 50.8 x 50.8 mm, 47 parts, among them J1 10118194-0001LF, J2 67996-412HLF, J3 Conn_01x06_Male, J4 Conn_01x06_Male, J5 Conn_01x06_Male, U1 AP2114H-3_3TRG1, U2 STM32L152RETx, U3 ESP-07, Y1 8MHz, Y2 SIT1533AI-H4-DCC-32_768E

Commit message: Routing complete
Parts:
- removed J2: 67996-412HLF, digikey-footprints:PinHeader_6x2_P2.54mm_Vertical
- BOOT1, BOOT2, C1, C12, C13, C14, C15, C2, C7, J1, J4, J5, R1, S1, S2, S3, S4, U1, U3, Y1: moved to F.Cu
- C10, C11, J3, R3, R4, R5, R6, R7: moved to B.Cu
- moved C16 109.7 mm to (143.5, 103.6)
- moved C3 88.0 mm to (116.5, 84.5)
- moved C10 80.0 mm to (117.1, 114.8), turned to 270 degrees
- moved C11 75.3 mm to (118.9, 114.8), turned to 270 degrees
- moved C9 74.9 mm to (108.7, 117.6), turned to 270 degrees
- moved S4 60.5 mm to (105.4, 122.3), turned to 90 degrees
- moved C15 56.6 mm to (105.4, 118.6)
- moved D4 44.9 mm to (149.9, 80.0), turned to 270 degrees
- moved J4 43.2 mm to (105.4, 108.0)
- moved J5 43.2 mm to (148.6, 95.2)
- moved D3 42.2 mm to (146.1, 80.0), turned to 270 degrees
- moved R7 41.1 mm to (149.9, 83.8), turned to 90 degrees
- moved D2 39.8 mm to (142.2, 80.0), turned to 270 degrees
- moved R6 38.5 mm to (146.1, 83.8), turned to 90 degrees
- moved D1 37.9 mm to (138.4, 80.0), turned to 270 degrees
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Connections:
- C12 pad 1: Net-(C12-Pad1) -> /BUTTON1
- C13 pad 1: Net-(C13-Pad1) -> /BUTTON2
- C14 pad 1: Net-(C14-Pad1) -> /BUTTON3
- C16 pad 2: VDD -> GND
- D1 pad 1: Net-(D1-Pad1) -> /LED1
- D2 pad 1: Net-(D2-Pad1) -> /LED2
- D3 pad 1: Net-(D3-Pad1) -> /LED3
- D4 pad 1: Net-(D4-Pad1) -> /LED4
- S1 pad 1: Net-(C12-Pad1) -> /BUTTON1
- S2 pad 1: Net-(C13-Pad1) -> /BUTTON2
- S3 pad 1: Net-(C14-Pad1) -> /BUTTON3
- U2 pad 10: /ESP_ENABLE -> (no net)
- U2 pad 11: /ESP_NRST -> (no net)
- U2 pad 14: Net-(D1-Pad1) -> (no net)
- U2 pad 15: Net-(D2-Pad1) -> (no net)
- U2 pad 16: Net-(D3-Pad1) -> (no net)
- U2 pad 17: Net-(D4-Pad1) -> (no net)
- U2 pad 20: (no net) -> /ESP_NRST
- U2 pad 21: (no net) -> /ESP_ENABLE
- U2 pad 22: (no net) -> /ESP_WAKE
- U2 pad 24: /ESP_WAKE -> (no net)
- U2 pad 26: (no net) -> /ESP_GPIO0
- U2 pad 27: (no net) -> /ESP_GPIO2
- U2 pad 28: /BOOT1 -> (no net)
- U2 pad 37: (no net) -> /BOOT1
- U2 pad 38: (no net) -> /BUTTON3
- U2 pad 39: (no net) -> /BUTTON2
- U2 pad 40: (no net) -> /BUTTON1
- U2 pad 41: (no net) -> /BOOT0
- U2 pad 56: (no net) -> /LED1
- U2 pad 57: Net-(C14-Pad1) -> /LED2
- U2 pad 58: Net-(C13-Pad1) -> /LED3
- U2 pad 59: Net-(C12-Pad1) -> /LED4
- U2 pad 60: /BOOT0 -> (no net)
- U2 pad 8: /ESP_GPIO0 -> (no net)
- U2 pad 9: /ESP_GPIO2 -> (no net)
Routing:
- net Net-(C12-Pad1): track 59.6 -> 0.00 mm, vias 1 -> 0
- net /LED4: track 0.00 -> 56.9 mm, vias 0 -> 1
- net /LED3: track 0.00 -> 52.5 mm, vias 0 -> 1
- net /LED2: track 0.00 -> 49.8 mm, vias 0 -> 1
- net Net-(C13-Pad1): track 49.4 -> 0.00 mm, vias 1 -> 0
- net /LED1: track 0.00 -> 47.1 mm, vias 0 -> 1
- net /~RESET: track 57.9 -> 13.8 mm
- net Net-(C14-Pad1): track 40.6 -> 0.00 mm, vias 1 -> 0
- net /BUTTON3: track 0.00 -> 35.8 mm
- net /BUTTON2: track 0.00 -> 33.8 mm
- net /BUTTON1: track 0.00 -> 32.4 mm
- net /I2C1_SDA: track 39.5 -> 68.4 mm, vias 1 -> 0
- net /I2C1_SCL: track 41.9 -> 70.4 mm
- net /SPI2_NSS: track 36.1 -> 8.94 mm, vias 1 -> 0
- net /BOOT1: track 47.8 -> 25.0 mm, vias 0 -> 1
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- added copper zone on F.Cu, net GND
- added copper zone on B.Cu, net VDD
- removed copper zone on B.Cu, net GND
- removed copper zone on F.Cu, net VDD
Other:
- net class Default: trace_width 0.1524 -> 0.2032
- net class Power: clearance 0.1524 -> 0.2032; trace_width 0.38608 -> 0.381
- net class Power-Decoupling added: clearance 0.1524, trace_width 0.2032, via_dia 0.6858, via_drill 0.3302
- board text added: "CLOCK3"
- board text removed: "HOURS"
- board text removed: "MINUTES"
- board text removed: "RESET"
- board text removed: "SECS"

Commit message: wip
Parts:
- removed C16: 1uF, Capacitor_SMD:C_0603_1608Metric
- removed R1: 390, Resistor_SMD:R_0603_1608Metric
- removed U3: ESP-07, RF_Module:ESP-07
- added BAT1: BS-7, digikey-footprints:Battery_Holder_Coin_2032_BS-7, F.Cu at (142.4, 115.3)
- added C17: 5pF, Capacitor_SMD:C_0603_1608Metric, F.Cu at (113.0, 111.7)
- added C18: 5pF, Capacitor_SMD:C_0603_1608Metric, F.Cu at (115.6, 111.8)
- added J2: SWD, Connector_Molex:Molex_KK-254_AE-6410-06A_1x06_P2.54mm_Vertical, F.Cu at (106.2, 123.4)
- C10: value 100nF -> 10nF; moved to F.Cu
- C11, R3: moved to F.Cu
- C4, C5: value 20pF -> 16pF; moved to B.Cu
- C9: value 100nF -> 4.7uF
- S1, S2, S3, S4: value B3U-1000P -> B3F-3150; footprint digikey-footprints:Switch_Tactile_SMD_B3U-1000P -> synack-common:B3F-3150
- U2: value STM32L152RETx -> STM32F102CBTx; footprint Package_QFP:LQFP-64_10x10mm_P0.5mm -> Package_QFP:LQFP-48_7x7mm_P0.5mm
- Y1: value 8MHz -> 8MHz 18pF 30ppm; footprint Crystal:Crystal_HC49-4H_Vertical -> synack-common:Crystal_SMD_HC49-US_AT49; moved to B.Cu
- Y2: value SIT1533AI-H4-DCC-32_768E -> 32.768kHz 12.5pF 20ppm; footprint digikey-footprints:Oscillator_MEMS_SIT1533AI-H4-DCC-32.768E -> Crystal:Crystal_SMD_SeikoEpson_MC146-4Pin_6.7x1.5mm
- moved U1 34.4 mm to (147.4, 80.0)
- moved C2 34.2 mm to (147.0, 84.5)
- moved C1 34.0 mm to (144.0, 84.5)
- moved C3 33.7 mm to (150.2, 84.5)
- moved D1 30.6 mm to (158.8, 57.1)
- moved D2 30.6 mm to (162.6, 57.1)
- moved D3 30.6 mm to (166.4, 57.1)
- moved D4 30.6 mm to (170.2, 57.1)
- moved R4 30.6 mm to (158.8, 61.0)
- moved R5 30.6 mm to (162.6, 61.0)
- moved R6 30.6 mm to (166.4, 61.0)
- moved R7 30.6 mm to (170.2, 61.0)
- moved S4 28.5 mm to (79.4, 110.8)
- moved BOOT1 26.9 mm to (138.4, 95.2)
- moved Y1 23.1 mm to (117.2, 101.6)
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Connections:
- C10 pad 1: GND -> VDD
- C10 pad 2: VDD -> GND
- C11 pad 1: GND -> VDD
- C11 pad 2: VDD -> GND
- C12 pad 1: /BUTTON1 -> GND
- C12 pad 2: GND -> /BUTTON1
- C13 pad 1: /BUTTON2 -> GND
- C13 pad 2: GND -> /BUTTON2
- C14 pad 1: /BUTTON3 -> GND
- C14 pad 2: GND -> /BUTTON3
- C15 pad 1: /~RESET -> GND
- C15 pad 2: GND -> /~RESET
- C6 pad 1: GND -> VDD
- C6 pad 2: VDD -> GND
- C7 pad 1: GND -> VDD
- C7 pad 2: VDD -> GND
- C8 pad 1: GND -> VDD
- C8 pad 2: VDD -> GND
- C9 pad 1: GND -> VDD
- C9 pad 2: VDD -> GND
- D4 pad 1: /LED4 -> (no net)
- MK3 pad 1: VDD -> GND
- MK4 pad 1: VDD -> GND
- S4 pad 1: GND -> /~RESET
- S4 pad 2: /~RESET -> GND
- U2 pad 1: (no net) -> /VBAT
- U2 pad 10: (no net) -> /LED1
- U2 pad 11: (no net) -> /LED2
- U2 pad 12: GND -> (no net)
- U2 pad 13: VDD -> (no net)
- U2 pad 18: GND -> (no net)
- U2 pad 19: VDD -> (no net)
- U2 pad 20: /ESP_NRST -> /BOOT1
- U2 pad 21: /ESP_ENABLE -> (no net)
- U2 pad 22: /ESP_WAKE -> (no net)
- U2 pad 23: (no net) -> GND
- U2 pad 24: (no net) -> VDD
- U2 pad 26: /ESP_GPIO0 -> /BUTTON3
- U2 pad 27: /ESP_GPIO2 -> /BUTTON2
- U2 pad 28: (no net) -> /BUTTON1
- U2 pad 29: /USART3_TX -> /LED3
- U2 pad 3: Net-(U2-Pad3) -> Net-(C17-Pad1)
- U2 pad 30: /USART3_RX -> (no net)
- U2 pad 31: GND -> (no net)
- U2 pad 32: VDD -> /USB_D-
- U2 pad 33: /SPI2_NSS -> /USB_D+
- U2 pad 34: /SPI2_SCK -> /SWDIO
- U2 pad 35: /SPI2_MISO -> GND
- U2 pad 36: /SPI2_MOSI -> VDD
- U2 pad 37: /BOOT1 -> /SWCLK
- U2 pad 38: /BUTTON3 -> (no net)
- U2 pad 39: /BUTTON2 -> /SWO
- U2 pad 4: (no net) -> Net-(C18-Pad1)
- U2 pad 40: /BUTTON1 -> (no net)
- U2 pad 41: /BOOT0 -> (no net)
- U2 pad 42: /USART1_TX -> /I2C1_SCL
- U2 pad 43: /USART1_RX -> /I2C1_SDA
- U2 pad 44: /USB_D- -> /BOOT0
- U2 pad 45: /USB_D+ -> (no net)
- U2 pad 46: /SWDIO -> (no net)
- U2 pad 6: Net-(R1-Pad1) -> Net-(C5-Pad1)
- U2 pad 8: (no net) -> GND
- U2 pad 9: (no net) -> VDD
- Y2 pad 1: (no net) -> Net-(C18-Pad1)
- Y2 pad 2: GND -> Net-(C17-Pad1)
- Y2 pad 3: Net-(U2-Pad3) -> (no net)
- Y2 pad 4: VDD -> (no net)
Routing:
- net VDD: track 111.7 -> 181.3 mm, vias 6 -> 0
- net /I2C1_SCL: track 70.4 -> 8.96 mm
- net /I2C1_SDA: track 68.4 -> 8.13 mm
- net /LED4: track 56.9 -> 0.00 mm, vias 1 -> 0
- net GND: track 65.2 -> 10.9 mm, vias 3 -> 0
- net /LED3: track 52.5 -> 0.00 mm, vias 1 -> 0
- net /LED2: track 49.8 -> 0.00 mm, vias 1 -> 0
- net VCC: track 88.4 -> 40.6 mm, vias 1 -> 0
- net /LED1: track 47.1 -> 0.00 mm, vias 1 -> 0
- net /SPI2_MOSI: track 29.4 -> 0.00 mm
- net /SWO: track 0.00 -> 28.9 mm, vias 0 -> 1
- net /SWDIO: track 0.00 -> 28.4 mm, vias 0 -> 1
- net /SWCLK: track 0.00 -> 28.0 mm, vias 0 -> 1
- net /SPI2_MISO: track 27.9 -> 0.00 mm, vias 2 -> 0
- net /SPI2_SCK: track 26.7 -> 0.00 mm
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- added copper zone on B.Cu, net GND
- added copper zone on F.Cu, net VDD
- removed copper zone on B.Cu, net VDD
