File: clock3.sch (KiCad schematic (older format))
At the start: 47 parts, among them J1 10118194-0001LF, J2 67996-412HLF, J3 Conn_01x06_Male, J4 Conn_01x06_Male, J5 Conn_01x06_Male, U1 AP2114H-3_3TRG1, U2 STM32L152RETx, U3 ESP-07, Y1 8MHz, Y2 SIT1533AI-H4-DCC-32_768E

Commit message: Routing complete
Connections:
- net labels added: BUTTON1, BUTTON2, BUTTON3, LED1, LED2, LED3, LED4
- wire segments 108 -> 104
- no-connect marks 26 -> 14
Other:
- note added: "LEDS"

Commit message: wip
Parts:
- removed C16: 1uF, Capacitor_SMD:C_0603_1608Metric, symbol Device:C
- removed C6: 100nF, Capacitor_SMD:C_0603_1608Metric, symbol Device:C
- removed J2: 67996-412HLF, digikey-footprints:PinHeader_6x2_P2.54mm_Vertical, symbol dk_Rectangular-Connectors-Headers-Male-Pins:67996-412HLF
- removed R1: 390, Resistor_SMD:R_0603_1608Metric, symbol Device:R
- removed S1, S2, S3, S4: B3U-1000P, digikey-footprints:Switch_Tactile_SMD_B3U-1000P, symbol dk_Tactile-Switches:B3U-1000P
- removed U2: STM32L152RETx, Package_QFP:LQFP-64_10x10mm_P0.5mm, symbol MCU_ST_STM32L1:STM32L152RETx
- removed U3: ESP-07, RF_Module:ESP-07, symbol RF_Module:ESP-07
- removed Y2: SIT1533AI-H4-DCC-32_768E, digikey-footprints:Oscillator_MEMS_SIT1533AI-H4-DCC-32.768E, symbol dk_Oscillators:SIT1533AI-H4-DCC-32_768E
- added BAT1: BS-7, digikey-footprints:Battery_Holder_Coin_2032_BS-7, symbol dk_Battery-Holders-Clips-Contacts:BS-7
- added C17, C18: 5pF, Capacitor_SMD:C_0603_1608Metric, symbol Device:C
- added C7: 100nF, Capacitor_SMD:C_0603_1608Metric, symbol Device:C
- added J2: SWD, Connector_Molex:Molex_KK-254_AE-6410-06A_1x06_P2.54mm_Vertical, symbol Connector_Generic:Conn_01x06
- added S1, S2, S3, S4: B3F-3150, synack-common:B3F-3150, symbol synack-common:B3F-3150
- added U2: STM32F102CBTx, Package_QFP:LQFP-48_7x7mm_P0.5mm, symbol MCU_ST_STM32F1:STM32F102CBTx
- added Y2: 32.768kHz 12.5pF 20ppm, Crystal:Crystal_SMD_SeikoEpson_MC146-4Pin_6.7x1.5mm, symbol Device:Crystal
- C10: value 100nF -> 10nF
- C4, C5: value 20pF -> 16pF
- C9: value 100nF -> 4.7uF
- Y1: value 8MHz -> 8MHz 18pF 30ppm; footprint Crystal:Crystal_HC49-4H_Vertical -> synack-common:Crystal_SMD_HC49-US_AT49
- renumbered C7 to C6
Connections:
- net labels added: VBAT
- net labels removed: 5VIN, ESP_ENABLE, ESP_GPIO0, ESP_GPIO2, ESP_NRST, ESP_WAKE, SPI2_MISO, SPI2_MOSI, SPI2_NSS, SPI2_SCK, USART1_RX, USART1_TX, USART3_RX, USART3_TX
- wire segments 104 -> 88
- no-connect marks 14 -> 8
Other:
- note added: "VDD3"
- note added: "VDDA"
